File: VESC6_OPEN_HARDWARE.kicad_pcb (KiCad board)
At the start: 4 copper layers, 110 x 45 mm, 131 parts, among them P1 USB_OTG, P10 PH_A, P11 SUPPLY, P12 GND, P2 CAN2, P3 SWD, P4 HALL/Encoder, P5 CAN1, P6 ADC_SWITCH, P8 PH_C, P9 PH_B, Q1 STL130N6F7, Q2 STL130N6F7, Q3 STL130N6F7, Q4 STL130N6F7, Q5 STL130N6F7, Q6 STL130N6F7, U1 STM32F40X_LQFP64, U10 LSM6DS3TR-C, U2 LM3671, U3 DRV8301, U4 TJA1051TK-3, U5 AD8418, U6 AD8418, U7 AD8418, X1 8m

Commit message: Release1
Parts:
- moved G*** 0.16 mm to (76.6, 41.6)
- renumbered P6 to ADC/SW, P5 to CAN, P2 to CAN, P4 to SENSE, P3 to SWD, P1 to USB
Routing:
- net SUPPLY: vias 2 -> 17
- added copper zone on In1.Cu, net SUPPLY
Changed lines of the file:
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@@
 			(drillshape 0)
 			(scaleselection 1)
-			(outputdirectory "FABRICATION/RELEASE1.1/")
+			(outputdirectory "FABRICATION/RELEASE1/")
 		)
 	)
@@
 			(at 10.597862 7.022693 0)
 			(layer "F.SilkS")
+			(hide yes)
 			(effects
 				(font
@@
 		(descr "JST SH series connector, SM06B-SRSS-TB (http://www.jst-mfg.com/product/pdf/eng/eSH.pdf), generated with kicad-footprint-generator")
 		(tags "connector JST SH horizontal")
-		(property "Reference" "P3"
+		(property "Reference" "SWD"
 			(at 0 -3.98 0)
 			(layer "F.SilkS")
@@
 			(pinfunction "Pin_1")
 			(pintype "passive")
-			(clearance 1)
+			(clearance 0)
 		)
 		(embedded_fonts no)
@@
 			(pinfunction "Pin_1")
 			(pintype "passive")
+			(clearance 1)
 		)
 		(embedded_fonts no)
@@
 		(descr "JST SH series connector, SM04B-SRSS-TB (http://www.jst-mfg.com/product/pdf/eng/eSH.pdf), generated with kicad-footprint-generator")
 		(tags "connector JST SH horizontal")
-		(property "Reference" "P5"
-			(at 0.09 -4.075 0)
+		(property "Reference" "CAN"
+			(at 0.08 -4.015 0)
 			(layer "F.SilkS")
 			(effects
@@
 		(tags "capacitor")
 		(property "Reference" "C14"
-			(at -1.16 1.45 90)
+			(at 3.045 0.03 90)
 			(layer "F.SilkS")
 			(effects
@@
 		(descr "Micro USB B receptable with flange, bottom-mount, SMD, right-angle (http://www.molex.com/pdm_docs/sd/473460001_sd.pdf)")
 		(tags "Micro B USB SMD")
-		(property "Reference" "P1"
+		(property "Reference" "USB"
 			(at 0 -3.3 0)
 			(layer "F.SilkS")
@@
 		(descr "JST SH series connector, SM04B-SRSS-TB (http://www.jst-mfg.com/product/pdf/eng/eSH.pdf), generated with kicad-footprint-generator")
 		(tags "connector JST SH horizontal")
-		(property "Reference" "P2"
-			(at -0.24 -3.735 0)
+		(property "Reference" "CAN"
+			(at -0.35 -3.985 0)
 			(layer "F.SilkS")
 			(effects
@@
 	(footprint "LOGO"
 		(layer "F.Cu")
-		(at 76.51 41.46)
+		(at 76.586265 41.603353)
 		(property "Reference" "G***"
 			(at 0 6.01 0)
 			(layer "F.SilkS")
+			(hide yes)
 			(effects
 				(font
@@
 		(descr "JST SH series connector, SM06B-SRSS-TB (http://www.jst-mfg.com/product/pdf/eng/eSH.pdf), generated with kicad-footprint-generator")
 		(tags "connector JST SH horizontal")
-		(property "Reference" "P4"
+		(property "Reference" "SENSE"
 			(at 0.02 -4.195 90)
 			(layer "F.SilkS")
@@
 			(pinfunction "Pin_1")
 			(pintype "passive")
+			(clearance 1)
 		)
 		(embedded_fonts no)
@@
 		(tags "capacitor")
 		(property "Reference" "C19"
-			(at -0.055 -1.43 90)
+			(at 3.13 -0.02 90)
 			(layer "F.SilkS")
 			(effects
@@
 		(descr "JST SH series connector, SM04B-SRSS-TB (http://www.jst-mfg.com/product/pdf/eng/eSH.pdf), generated with kicad-footprint-generator")
 		(tags "connector JST SH horizontal")
-		(property "Reference" "P6"
-			(at 0 -3.98 0)
+		(property "Reference" "ADC/SW"
+			(at 0.01 -3.965 0)
 			(layer "F.SilkS")
 			(effects
@@
 	)
 	(gr_text "Designed by Craig Gault\ngithub.com/craigg96"
-		(at 0.85 42.71 -0)
+		(at 0.82 42.83 -0)
 		(layer "F.SilkS")
 		(effects
@@
 	)
 	(via
+		(at 27.61 28.51)
+		(size 0.8)
+		(drill 0.4)
+		(layers "F.Cu" "B.Cu")
+		(free yes)
+		(net 23)
+	)
+	(via
+		(at 29.83 28.54)
+		(size 0.8)
+		(drill 0.4)
+		(layers "F.Cu" "B.Cu")
+		(free yes)
+		(net 23)
+	)
+	(via
+		(at 32.05 18.54)
+		(size 0.8)
+		(drill 0.4)
+		(layers "F.Cu" "B.Cu")
+		(free yes)
+		(net 23)
+	)
+	(via
+		(at 28.7 28.54)
+		(size 0.8)
+		(drill 0.4)
+		(layers "F.Cu" "B.Cu")
+		(free yes)
+		(net 23)
+	)
+	(via
+		(at 32.05 28.55)
+		(size 0.8)
+		(drill 0.4)
+		(layers "F.Cu" "B.Cu")
+		(free yes)
+		(net 23)
+	)
+	(via
+		(at 28.43 41.82)
+		(size 0.8)
+		(drill 0.4)
+		(layers "F.Cu" "B.Cu")
+		(free yes)
+		(net 23)
+	)
+	(via
+		(at 28.44 39.6)
+		(size 0.8)
+		(drill 0.4)
+		(layers "F.Cu" "B.Cu")
+		(free yes)
+		(net 23)
+	)
+	(via
+		(at 28.4 44.04)
+		(size 0.8)
+		(drill 0.4)
+		(layers "F.Cu" "B.Cu")
+		(free yes)
+		(net 23)
+	)
+	(via
+		(at 31 18.54)
+		(size 0.8)
+		(drill 0.4)
+		(layers "F.Cu" "B.Cu")
+		(free yes)
+		(net 23)
+	)
+	(via
+		(at 28.44 40.65)
+		(size 0.8)
+		(drill 0.4)
+		(layers "F.Cu" "B.Cu")
+		(free yes)
+		(net 23)
+	)
+	(via
 		(at 56.05 37.7)
 		(size 0.8)
@@
 		(net 23)
 	)
+	(via
+		(at 27.61 18.5)
+		(size 0.8)
+		(drill 0.4)
+		(layers "F.Cu" "B.Cu")
+		(free yes)
+		(net 23)
+	)
+	(via
+		(at 28.7 18.53)
+		(size 0.8)
+		(drill 0.4)
+		(layers "F.Cu" "B.Cu")
+		(free yes)
+		(net 23)
+	)
+	(via
+		(at 28.43 42.95)
+		(size 0.8)
+		(drill 0.4)
+		(layers "F.Cu" "B.Cu")
+		(free yes)
+		(net 23)
+	)
+	(via
+		(at 29.83 18.53)
+		(size 0.8)
+		(drill 0.4)
+		(layers "F.Cu" "B.Cu")
+		(free yes)
+		(net 23)
+	)
+	(via
+		(at 31 28.55)
+		(size 0.8)
+		(drill 0.4)
+		(layers "F.Cu" "B.Cu")
+		(free yes)
+		(net 23)
+	)
 	(segment
 		(start 56.05 37.7)
@@
 	)
 	(zone
-		(net 21)
-		(net_name "/DRV8301/SH_C")
+		(net 0)
+		(net_name "")
 		(layer "F.Cu")
 		(hatch edge 0.5)
-		(priority 2)
 		(connect_pads yes
 			(clearance 0)
@@
 		(min_thickness 0.25)
 		(filled_areas_thickness no)
-		(fill yes
-			(thermal_gap 0.5)
-			(thermal_bridge_width 0.5)
+		(keepout
+			(tracks allowed)
+			(vias allowed)
+			(pads allowed)
+			(copperpour not_allowed)
+			(footprints allowed)
+		)
+		(placement
+			(enabled no)
+			(sheetname "")
 		)
-		(polygon
-			(pts
-				(xy 19.34 11.719391) (xy 19.34 15.319391) (xy 17.44 15.319391) (xy 17.44 11.719391)
-			)
-		)
-	)
-	(zone
-		(net 107)
-		(net_name "Net-(P9-Pin_1)")
-		(layer "F.Cu")
-		(hatch edge 0.5)
-		(priority 1)
-		(connect_pads yes
-			(clearance 0)
-		)
-		(min_thickness 0.25)
-		(filled_areas_thickness no)
-		(fill yes
+		(fill
 			(thermal_gap 0.5)
 			(thermal_bridge_width 0.5)
@@
 		(polygon
 			(pts
-				(xy 10.215 21.69) (xy 1.056548 21.69) (xy 1.079817 25.32) (xy 10.215 25.32)
+				(xy 109.881659 8.7) (xy 106.296666 8.7) (xy 104.88 9.95) (xy 104.89 12.52) (xy 106.293188 13.66546)
+				(xy 109.891266 13.702048)
 			)
 		)
@@
 		(hatch edge 0.5)
 		(priority 2)
-		(connect_pads
+		(connect_pads yes
 			(clearance 0)
 		)
@@
 		(polygon
 			(pts
-				(xy 25.89 12.219391) (xy 25.89 15.519391) (xy 22.89 15.519391) (xy 22.89 12.219391)
+				(xy 19.34 11.719391) (xy 19.34 15.319391) (xy 17.44 15.319391) (xy 17.44 11.719391)
 			)
 		)
 	)
 	(zone
-		(net 23)
-		(net_name "SUPPLY")
+		(net 107)
+		(net_name "Net-(P9-Pin_1)")
 		(layer "F.Cu")
 		(hatch edge 0.5)
-		(priority 4)
+		(priority 1)
 		(connect_pads yes
 			(clearance 0)
@@
 		(polygon
 			(pts
-				(xy 27.0375 11.563782) (xy 27.0375 44.713782) (xy 32.9425 44.713782) (xy 32.9425 11.563782)
+				(xy 10.215 21.69) (xy 1.056548 21.69) (xy 1.079817 25.32) (xy 10.215 25.32)
 			)
 		)
 	)
 	(zone
-		(net 23)
-		(net_name "SUPPLY")
+		(net 21)
+		(net_name "/DRV8301/SH_C")
 		(layer "F.Cu")
 		(hatch edge 0.5)
-		(priority 4)
-		(connect_pads yes
+		(priority 2)
+		(connect_pads
 			(clearance 0)
 		)
 		(min_thickness 0.25)
 		(filled_areas_thickness no)
-		(fill
+		(fill yes
 			(thermal_gap 0.5)
 			(thermal_bridge_width 0.5)
@@
 		(polygon
 			(pts
-				(xy 31.623782 44.715) (xy 109.732409 44.715) (xy 109.805193 0.190729) (xy 98.41 0.37) (xy 98.495 32.355)
-				(xy 96.605 34.315) (xy 81.341572 34.315) (xy 77.609272 38.446477) (xy 31.623782 38.3)
+				(xy 25.89 12.219391) (xy 25.89 15.519391) (xy 22.89 15.519391) (xy 22.89 12.219391)
 			)
 		)
@@
 			)
 		)
+	)
+	(zone
+		(net 23)
+		(net_name "SUPPLY")
+		(layers "F.Cu" "In1.Cu")
+		(hatch edge 0.5)
+		(priority 4)
+		(connect_pads yes
+			(clearance 0)
+		)
+		(min_thickness 0.25)
+		(filled_areas_thickness no)
+		(fill yes
+			(thermal_gap 0.5)
+			(thermal_bridge_width 0.5)
+		)
+		(polygon
+			(pts
+				(xy 27.0375 11.563782) (xy 27.0375 44.713782) (xy 32.9425 44.713782) (xy 32.9425 11.563782)
+			)
+		)
+	)
+	(zone
+		(net 23)
+		(net_name "SUPPLY")
+		(layers "F.Cu" "In1.Cu")
+		(hatch edge 0.5)
+		(priority 4)
+		(connect_pads yes
+			(clearance 0)
+		)
+		(min_thickness 0.25)
+		(filled_areas_thickness no)
+		(fill yes
+			(thermal_gap 0.5)
+			(thermal_bridge_width 0.5)
+		)
+		(polygon
+			(pts
+				(xy 31.623782 44.715) (xy 109.732409 44.715) (xy 109.805193 0.190729) (xy 98.41 0.23) (xy 98.495 32.355)
+				(xy 96.605 34.315) (xy 81.341572 34.315) (xy 77.609272 38.446477) (xy 31.623782 38.3)
+			)
+		)
