File: power.kicad_sch (KiCad schematic)
At the start: 45 parts, among them P10 PH_A, P11 SUPPLY, P12 GND, P8 PH_C, P9 PH_B, Q1 STL130N6F7, Q2 STL130N6F7, Q3 STL130N6F7, Q4 STL130N6F7, Q5 STL130N6F7, Q6 STL130N6F7, U5 AD8418, U6 AD8418, U7 AD8418

Commit message: Finished routing
Parts:
- C37, C39, C40, C41, C43, C44: LCSC part no. C385986 -> C385987
Changed lines of the file:
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@@
 			)
 		)
-		(property "LCSC part no." "C385986"
+		(property "LCSC part no." "C385987"
 			(at 181.61 63.5 0)
 			(effects
@@
 			)
 		)
-		(property "LCSC part no." "C385986"
+		(property "LCSC part no." "C385987"
 			(at 190.5 63.5 0)
 			(effects
@@
 			)
 		)
-		(property "LCSC part no." "C385986"
+		(property "LCSC part no." "C385987"
 			(at 87.63 64.77 0)
 			(effects
@@
 			)
 		)
-		(property "LCSC part no." "C385986"
+		(property "LCSC part no." "C385987"
 			(at 96.52 64.77 0)
 			(effects
@@
 			)
 		)
-		(property "LCSC part no." "C385986"
+		(property "LCSC part no." "C385987"
 			(at 269.24 64.77 0)
 			(effects
@@
 			)
 		)
-		(property "LCSC part no." "C385986"
+		(property "LCSC part no." "C385987"
 			(at 278.13 64.77 0)
 			(effects

Commit message: drc clear, added images
Parts:
- P11, P12: footprint Connector_Pin:Pin_D1.0mm_L10.0mm_LooseFit -> Connector_Pin:Pin_D1.3mm_L11.0mm_LooseFit
Changed lines of the file:
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@@
 			)
 		)
-		(property "Footprint" "Connector_Pin:Pin_D1.0mm_L10.0mm_LooseFit"
+		(property "Footprint" "Connector_Pin:Pin_D1.3mm_L11.0mm_LooseFit"
 			(at 262.89 27.94 0)
 			(effects
@@
 			)
 		)
-		(property "Footprint" "Connector_Pin:Pin_D1.0mm_L10.0mm_LooseFit"
+		(property "Footprint" "Connector_Pin:Pin_D1.3mm_L11.0mm_LooseFit"
 			(at 271.78 107.95 0)
 			(effects

Commit message: Release1
Parts:
- C37, C39, C40, C41, C43, C44: Link https://jlcpcb.com/partdetail/TaiyoYuden-HMK325C7475KMHPE/C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 -> (none); MFP HMK325C7475KMHPE -> (none)
- C48, C49, C50, C51: Link https://jlcpcb.com/partdetail/Nichicon-URZ1J221MHD/C433278 -> (none); MFP URZ1J221MHD -> (none)
Changed lines of the file:
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@@
 			)
 		)
-		(property "Datasheet" "https://datasheet.lcsc.com/lcsc/2211282230_Taiyo-Yuden-HMK325C7475KMHPE_C385986.pdf"
+		(property "Datasheet" ""
 			(at 181.61 63.5 0)
 			(effects
@@
 			)
 		)
-		(property "Link" "https://jlcpcb.com/partdetail/TaiyoYuden-HMK325C7475KMHPE/C385986"
+		(property "Link" ""
 			(at 181.61 63.5 0)
 			(effects
@@
 			)
 		)
-		(property "MFP" "HMK325C7475KMHPE"
+		(property "MFP" ""
 			(at 181.61 63.5 0)
 			(effects
@@
 			)
 		)
-		(property "Datasheet" "https://datasheet.lcsc.com/lcsc/2211282230_Taiyo-Yuden-HMK325C7475KMHPE_C385986.pdf"
+		(property "Datasheet" ""
 			(at 190.5 63.5 0)
 			(effects
@@
 			)
 		)
-		(property "Link" "https://jlcpcb.com/partdetail/TaiyoYuden-HMK325C7475KMHPE/C385986"
+		(property "Link" ""
 			(at 190.5 63.5 0)
 			(effects
@@
 			)
 		)
-		(property "MFP" "HMK325C7475KMHPE"
+		(property "MFP" ""
 			(at 190.5 63.5 0)
 			(effects
@@
 			)
 		)
-		(property "Datasheet" "https://datasheet.lcsc.com/lcsc/2211282230_Taiyo-Yuden-HMK325C7475KMHPE_C385986.pdf"
+		(property "Datasheet" ""
 			(at 87.63 64.77 0)
 			(effects
@@
 			)
 		)
-		(property "Link" "https://jlcpcb.com/partdetail/TaiyoYuden-HMK325C7475KMHPE/C385986"
+		(property "Link" ""
 			(at 87.63 64.77 0)
 			(effects
@@
 			)
 		)
-		(property "MFP" "HMK325C7475KMHPE"
+		(property "MFP" ""
 			(at 87.63 64.77 0)
 			(effects
@@
 			)
 		)
-		(property "Datasheet" "https://datasheet.lcsc.com/lcsc/2211282230_Taiyo-Yuden-HMK325C7475KMHPE_C385986.pdf"
+		(property "Datasheet" ""
 			(at 96.52 64.77 0)
 			(effects
@@
 			)
 		)
-		(property "Link" "https://jlcpcb.com/partdetail/TaiyoYuden-HMK325C7475KMHPE/C385986"
+		(property "Link" ""
 			(at 96.52 64.77 0)
 			(effects
@@
 			)
 		)
-		(property "MFP" "HMK325C7475KMHPE"
+		(property "MFP" ""
 			(at 96.52 64.77 0)
 			(effects
@@
 			)
 		)
-		(property "Datasheet" "https://datasheet.lcsc.com/lcsc/2211282230_Taiyo-Yuden-HMK325C7475KMHPE_C385986.pdf"
+		(property "Datasheet" ""
 			(at 269.24 64.77 0)
 			(effects
@@
 			)
 		)
-		(property "Link" "https://jlcpcb.com/partdetail/TaiyoYuden-HMK325C7475KMHPE/C385986"
+		(property "Link" ""
 			(at 269.24 64.77 0)
 			(effects
@@
 			)
 		)
-		(property "MFP" "HMK325C7475KMHPE"
+		(property "MFP" ""
 			(at 269.24 64.77 0)
 			(effects
@@
 			)
 		)
-		(property "Datasheet" "https://datasheet.lcsc.com/lcsc/2211282230_Taiyo-Yuden-HMK325C7475KMHPE_C385986.pdf"
+		(property "Datasheet" ""
 			(at 278.13 64.77 0)
 			(effects
@@
 			)
 		)
-		(property "Link" "https://jlcpcb.com/partdetail/TaiyoYuden-HMK325C7475KMHPE/C385986"
+		(property "Link" ""
 			(at 278.13 64.77 0)
 			(effects
@@
 			)
 		)
-		(property "MFP" "HMK325C7475KMHPE"
+		(property "MFP" ""
 			(at 278.13 64.77 0)
 			(effects
@@
 			)
 		)
-		(property "Datasheet" "~"
+		(property "Datasheet" ""
 			(at 19.05 55.88 0)
 			(effects
@@
 			)
 		)
-		(property "Datasheet" "~"
+		(property "Datasheet" ""
 			(at 113.03 54.61 0)
 			(effects
@@
 			)
 		)
-		(property "Datasheet" "~"
+		(property "Datasheet" ""
 			(at 200.66 55.88 0)
 			(effects
@@
 			)
 		)
-		(property "Datasheet" "~"
+		(property "Datasheet" ""
 			(at 262.89 27.94 0)
 			(effects
@@
 			)
 		)
-		(property "Datasheet" "~"
+		(property "Datasheet" ""
 			(at 271.78 107.95 0)
 			(effects
@@
 			)
 		)
-		(property "Datasheet" "https://www.farnell.com/datasheets/2815981.pdf"
+		(property "Datasheet" ""
 			(at 76.2 41.91 0)
 			(effects
@@
 			)
 		)
-		(property "Datasheet" "https://www.farnell.com/datasheets/2815981.pdf"
+		(property "Datasheet" ""
 			(at 76.2 82.55 0)
 			(effects
@@
 			)
 		)
-		(property "Datasheet" "https://www.farnell.com/datasheets/2815981.pdf"
+		(property "Datasheet" ""
 			(at 170.18 40.64 0)
 			(effects
@@
 			)
 		)
-		(property "Datasheet" "https://www.farnell.com/datasheets/2815981.pdf"
+		(property "Datasheet" ""
 			(at 170.18 81.28 0)
 			(effects
@@
 			)
 		)
-		(property "Datasheet" "https://www.farnell.com/datasheets/2815981.pdf"
+		(property "Datasheet" ""
 			(at 257.81 82.55 0)
 			(effects
@@
 			)
 		)
-		(property "Datasheet" "https://www.farnell.com/datasheets/2815981.pdf"
+		(property "Datasheet" ""
 			(at 257.81 41.91 0)
 			(effects
@@
 			)
 		)
-		(property "Datasheet" "https://datasheet.lcsc.com/lcsc/1912111437_Nichicon-URZ1J221MHD_C433278.pdf"
+		(property "Datasheet" ""
 			(at 238.76 135.89 0)
 			(effects
@@
 			)
 		)
-		(property "Link" "https://jlcpcb.com/partdetail/Nichicon-URZ1J221MHD/C433278"
+		(property "Link" ""
 			(at 238.76 135.89 0)
 			(effects
@@
 			)
 		)
-		(property "MFP" "URZ1J221MHD"
+		(property "MFP" ""
 			(at 238.76 135.89 0)
 			(effects
@@
 			)
 		)
-		(property "Datasheet" "https://datasheet.lcsc.com/lcsc/1912111437_Nichicon-URZ1J221MHD_C433278.pdf"
+		(property "Datasheet" ""
 			(at 226.06 135.89 0)
 			(effects
@@
 			)
 		)
-		(property "Link" "https://jlcpcb.com/partdetail/Nichicon-URZ1J221MHD/C433278"
+		(property "Link" ""
 			(at 226.06 135.89 0)
 			(effects
@@
 			)
 		)
-		(property "MFP" "URZ1J221MHD"
+		(property "MFP" ""
 			(at 226.06 135.89 0)
 			(effects
@@
 			)
 		)
-		(property "Datasheet" "https://datasheet.lcsc.com/lcsc/1912111437_Nichicon-URZ1J221MHD_C433278.pdf"
+		(property "Datasheet" ""
 			(at 250.19 135.89 0)
 			(effects
@@
 			)
 		)
-		(property "Link" "https://jlcpcb.com/partdetail/Nichicon-URZ1J221MHD/C433278"
+		(property "Link" ""
 			(at 250.19 135.89 0)
 			(effects
@@
 			)
 		)
-		(property "MFP" "URZ1J221MHD"
+		(property "MFP" ""
 			(at 250.19 135.89 0)
 			(effects
@@
 			)
 		)
-		(property "Datasheet" "https://datasheet.lcsc.com/lcsc/1912111437_Nichicon-URZ1J221MHD_C433278.pdf"
+		(property "Datasheet" ""
 			(at 262.89 135.89 0)
 			(effects
@@
 			)
 		)
-		(property "Link" "https://jlcpcb.com/partdetail/Nichicon-URZ1J221MHD/C433278"
+		(property "Link" ""
 			(at 262.89 135.89 0)
 			(effects
@@
 			)
 		)
-		(property "MFP" "URZ1J221MHD"
+		(property "MFP" ""
 			(at 262.89 135.89 0)
 			(effects

Commit message: publish
Parts:
- P10, P11, P12, P8, P9: LCSC part no. (none) -> C7200700
Changed lines of the file:
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@@
+			)
+		)
+		(property "LCSC part no." "C7200700"
+			(at 19.05 55.88 0)
+			(effects
+				(font
+					(size 1.27 1.27)
+				)
 			)
 		)
@@
 			)
 		)
+		(property "LCSC part no." "C7200700 "
+			(at 113.03 54.61 0)
+			(effects
+				(font
+					(size 1.27 1.27)
+				)
+			)
+		)
 		(pin "1"
 		)
@@
 			)
 		)
+		(property "LCSC part no." "C7200700 "
+			(at 200.66 55.88 0)
+			(effects
+				(font
+					(size 1.27 1.27)
+				)
+			)
+		)
 		(pin "1"
 		)
@@
 			)
 		)
+		(property "LCSC part no." "C7200700 "
+			(at 262.89 27.94 0)
+			(effects
+				(font
+					(size 1.27 1.27)
+				)
+			)
+		)
 		(pin "1"
 		)
@@
 			)
 		)
+		(property "LCSC part no." "C7200700 "
+			(at 271.78 107.95 0)
+			(effects
+				(font
+					(size 1.27 1.27)
+				)
+			)
+		)
